Commit message: feat: IV2023 demo
Signed-off-by: Amadeusz Szymko <amadeusz.szymko@put.poznan.pl>

File: f1tenth_sensor_kit_description/urdf/sensor_kit.xacro (robot description, xacro)
@@ -19,5 +19,5 @@
     <xacro:property name="calibration" value="${xacro.load_yaml('$(arg config_dir)/sensor_kit_calibration.yaml')}"/>
     <!-- lidar -->
-    <joint name="laser_joint" type="fixed">
+    <!-- <joint name="laser_joint" type="fixed">
       <origin
         xyz="${calibration['sensor_kit_base_link']['laser']['x']}
@@ -31,5 +31,5 @@
       <child link="laser"/>
     </joint>
-    <link name="laser"/>
+    <link name="laser"/> -->
     <!-- camera -->
     <joint name="camera_joint" type="fixed">

File: f1tenth_sensor_kit_description/urdf/sensors.xacro (robot description, xacro)
@@ -2,15 +2,15 @@
 <robot name="vehicle" xmlns:xacro="http://ros.org/wiki/xacro">
   <xacro:arg name="config_dir" default="$(find f1tenth_sensor_kit_description)/config"/>
-  <xacro:property name="calibration" value="${xacro.load_yaml('$(arg config_dir)/sensors_calibration.yaml')}"/>
+  <xacro:property name="calibartion" value="${xacro.load_yaml('$(arg config_dir)/sensors_calibration.yaml')}"/>
   <!-- sensor kit -->
   <xacro:include filename="sensor_kit.xacro"/>
   <xacro:sensor_kit_macro
     parent="base_link"
-    x="${calibration['base_link']['sensor_kit_base_link']['x']}"
-    y="${calibration['base_link']['sensor_kit_base_link']['y']}"
-    z="${calibration['base_link']['sensor_kit_base_link']['z']}"
-    roll="${calibration['base_link']['sensor_kit_base_link']['roll']}"
-    pitch="${calibration['base_link']['sensor_kit_base_link']['pitch']}"
-    yaw="${calibration['base_link']['sensor_kit_base_link']['yaw']}"
+    x="${calibartion['base_link']['sensor_kit_base_link']['x']}"
+    y="${calibartion['base_link']['sensor_kit_base_link']['y']}"
+    z="${calibartion['base_link']['sensor_kit_base_link']['z']}"
+    roll="${calibartion['base_link']['sensor_kit_base_link']['roll']}"
+    pitch="${calibartion['base_link']['sensor_kit_base_link']['pitch']}"
+    yaw="${calibartion['base_link']['sensor_kit_base_link']['yaw']}"
   />
 </robot>
